File: Hardware/VNA/gainPhaseDetect.sch (KiCad schematic (older format))
At the start: 27 parts, among them U12 PE4257, U13 AD8302

Commit message: added footprints and 3d models
Parts:
- C48, C49, C50, C51, C52, C55: footprint (none) -> Capacitor_SMD:C_0402_1005Metric
- R26, R27, R28, R29, R30, R31, R32, R33, R34, R35, R36: footprint (none) -> Resistor_SMD:R_0402_1005Metric
- R37, R38, R39, R40, R41: footprint (none) -> Resistor_SMD:R_0603_1608Metric
- U12: footprint (none) -> VNA_Footprints:QFN-20-1EP_4x4mm_P0.5mm_EP2.15x2.15mm_ThermalVias
- U13: footprint (none) -> Package_SO:TSSOP-14_4.4x5mm_P0.65mm
Changed lines of the file:
@@
 F 0 "U12" H 4000 2750 50  0000 C CNN
 F 1 "PE4257" H 4100 2650 50  0000 C CNN
-F 2 "" H 4650 3250 50  0001 C CNN
+F 2 "VNA_Footprints:QFN-20-1EP_4x4mm_P0.5mm_EP2.15x2.15mm_ThermalVias" H 4650 3250 50  0001 C CNN
 F 3 "" H 4650 3250 50  0001 C CNN
 	1    4650 3250
@@
 F 0 "R30" V 2350 4000 50  0000 C CNN
 F 1 "37R" V 2550 4000 50  0000 C CNN
-F 2 "" V 2380 4000 50  0001 C CNN
+F 2 "Resistor_SMD:R_0402_1005Metric" V 2380 4000 50  0001 C CNN
 F 3 "~" H 2450 4000 50  0001 C CNN
 	1    2450 4000
@@
 F 0 "R27" H 2270 4296 50  0000 L CNN
 F 1 "150R" H 2270 4205 50  0000 L CNN
-F 2 "" V 2130 4250 50  0001 C CNN
+F 2 "Resistor_SMD:R_0402_1005Metric" V 2130 4250 50  0001 C CNN
 F 3 "~" H 2200 4250 50  0001 C CNN
 	1    2200 4250
@@
 $EndComp
 $Comp
-L power:GND #PWR0101
+L power:GND #PWR066
 U 1 1 5CDA106C
 P 2700 4450
-F 0 "#PWR0101" H 2700 4200 50  0001 C CNN
+F 0 "#PWR066" H 2700 4200 50  0001 C CNN
 F 1 "GND" H 2705 4277 50  0000 C CNN
 F 2 "" H 2700 4450 50  0001 C CNN
@@
 $EndComp
 $Comp
-L power:GND #PWR0102
+L power:GND #PWR063
 U 1 1 5CDA1618
 P 2200 4450
-F 0 "#PWR0102" H 2200 4200 50  0001 C CNN
+F 0 "#PWR063" H 2200 4200 50  0001 C CNN
 F 1 "GND" H 2205 4277 50  0000 C CNN
 F 2 "" H 2200 4450 50  0001 C CNN
@@
 F 0 "R31" V 2350 5000 50  0000 C CNN
 F 1 "278R" V 2550 5000 50  0000 C CNN
-F 2 "" V 2380 5000 50  0001 C CNN
+F 2 "Resistor_SMD:R_0402_1005Metric" V 2380 5000 50  0001 C CNN
 F 3 "~" H 2450 5000 50  0001 C CNN
 	1    2450 5000
@@
 F 0 "R34" H 2770 5296 50  0000 L CNN
 F 1 "60R" H 2770 5205 50  0000 L CNN
-F 2 "" V 2630 5250 50  0001 C CNN
+F 2 "Resistor_SMD:R_0402_1005Metric" V 2630 5250 50  0001 C CNN
 F 3 "~" H 2700 5250 50  0001 C CNN
 	1    2700 5250
@@
 $EndComp
 $Comp
-L power:GND #PWR0103
+L power:GND #PWR067
 U 1 1 5CDA434F
 P 2700 5450
-F 0 "#PWR0103" H 2700 5200 50  0001 C CNN
+F 0 "#PWR067" H 2700 5200 50  0001 C CNN
 F 1 "GND" H 2705 5277 50  0000 C CNN
 F 2 "" H 2700 5450 50  0001 C CNN
@@
 $EndComp
 $Comp
-L power:GND #PWR0104
+L power:GND #PWR064
 U 1 1 5CDA4355
 P 2200 5450
-F 0 "#PWR0104" H 2200 5200 50  0001 C CNN
+F 0 "#PWR064" H 2200 5200 50  0001 C CNN
 F 1 "GND" H 2205 5277 50  0000 C CNN
 F 2 "" H 2200 5450 50  0001 C CNN
@@
 F 0 "R28" H 2270 5296 50  0000 L CNN
 F 1 "60R" H 2270 5205 50  0000 L CNN
-F 2 "" V 2130 5250 50  0001 C CNN
+F 2 "Resistor_SMD:R_0402_1005Metric" V 2130 5250 50  0001 C CNN
 F 3 "~" H 2200 5250 50  0001 C CNN
 	1    2200 5250
@@
 $EndComp
 $Comp
-L power:GND #PWR0105
+L power:GND #PWR069
 U 1 1 5CDB0BF2
 P 5450 5000
-F 0 "#PWR0105" H 5450 4750 50  0001 C CNN
+F 0 "#PWR069" H 5450 4750 50  0001 C CNN
 F 1 "GND" H 5455 4827 50  0000 C CNN
 F 2 "" H 5450 5000 50  0001 C CNN
@@
 F 0 "R29" V 2350 3050 50  0000 C CNN
 F 1 "0R0" V 2550 3050 50  0000 C CNN
-F 2 "" V 2380 3050 50  0001 C CNN
+F 2 "Resistor_SMD:R_0402_1005Metric" V 2380 3050 50  0001 C CNN
 F 3 "~" H 2450 3050 50  0001 C CNN
 	1    2450 3050
@@
 F 0 "R32" H 2770 3346 50  0000 L CNN
 F 1 "DNP" H 2770 3255 50  0000 L CNN
-F 2 "" V 2630 3300 50  0001 C CNN
+F 2 "Resistor_SMD:R_0402_1005Metric" V 2630 3300 50  0001 C CNN
 F 3 "~" H 2700 3300 50  0001 C CNN
 	1    2700 3300
@@
 $EndComp
 $Comp
-L power:GND #PWR0106
+L power:GND #PWR065
 U 1 1 5CDB41BA
 P 2700 3500
-F 0 "#PWR0106" H 2700 3250 50  0001 C CNN
+F 0 "#PWR065" H 2700 3250 50  0001 C CNN
 F 1 "GND" H 2705 3327 50  0000 C CNN
 F 2 "" H 2700 3500 50  0001 C CNN
@@
 $EndComp
 $Comp
-L power:GND #PWR0107
+L power:GND #PWR062
 U 1 1 5CDB41C0
 P 2200 3500
-F 0 "#PWR0107" H 2200 3250 50  0001 C CNN
+F 0 "#PWR062" H 2200 3250 50  0001 C CNN
 F 1 "GND" H 2205 3327 50  0000 C CNN
 F 2 "" H 2200 3500 50  0001 C CNN
@@
 $EndComp
 $Comp
-L power:GND #PWR0108
+L power:GND #PWR068
 U 1 1 5CDB9513
 P 4950 3650
-F 0 "#PWR0108" H 4950 3400 50  0001 C CNN
+F 0 "#PWR068" H 4950 3400 50  0001 C CNN
 F 1 "GND" H 4955 3477 50  0000 C CNN
 F 2 "" H 4950 3650 50  0001 C CNN
@@
 F 0 "R26" H 2270 3346 50  0000 L CNN
 F 1 "DNP" H 2270 3255 50  0000 L CNN
-F 2 "" V 2130 3300 50  0001 C CNN
+F 2 "Resistor_SMD:R_0402_1005Metric" V 2130 3300 50  0001 C CNN
 F 3 "~" H 2200 3300 50  0001 C CNN
 	1    2200 3300
@@
 F 0 "C52" H 8315 4596 50  0000 L CNN
 F 1 "DNP" H 8315 4505 50  0000 L CNN
-F 2 "" H 8238 4400 50  0001 C CNN
+F 2 "Capacitor_SMD:C_0402_1005Metric" H 8238 4400 50  0001 C CNN
 F 3 "~" H 8200 4550 50  0001 C CNN
 	1    8200 4550
@@
 F 0 "C55" H 8715 4596 50  0000 L CNN
 F 1 "DNP" H 8715 4505 50  0000 L CNN
-F 2 "" H 8638 4400 50  0001 C CNN
+F 2 "Capacitor_SMD:C_0402_1005Metric" H 8638 4400 50  0001 C CNN
 F 3 "~" H 8600 4550 50  0001 C CNN
 	1    8600 4550
@@
 $EndComp
 $Comp
-L power:GND #PWR0109
+L power:GND #PWR071
 U 1 1 5CEA8859
 P 7950 4400
-F 0 "#PWR0109" H 7950 4150 50  0001 C CNN
+F 0 "#PWR071" H 7950 4150 50  0001 C CNN
 F 1 "GND" H 7955 4227 50  0000 C CNN
 F 2 "" H 7950 4400 50  0001 C CNN
@@
 $EndComp
 $Comp
-L power:GND #PWR0110
+L power:GND #PWR072
 U 1 1 5CEA8E03
 P 8200 4800
-F 0 "#PWR0110" H 8200 4550 50  0001 C CNN
+F 0 "#PWR072" H 8200 4550 50  0001 C CNN
 F 1 "GND" H 8205 4627 50  0000 C CNN
 F 2 "" H 8200 4800 50  0001 C CNN
@@
 $EndComp
 $Comp
-L power:GND #PWR0111
+L power:GND #PWR074
 U 1 1 5CEA91AC
 P 8600 4800
-F 0 "#PWR0111" H 8600 4550 50  0001 C CNN
+F 0 "#PWR074" H 8600 4550 50  0001 C CNN
 F 1 "GND" H 8605 4627 50  0000 C CNN
 F 2 "" H 8600 4800 50  0001 C CNN
@@
 F 0 "R39" V 9450 2800 50  0000 C CNN
 F 1 "0R0" V 9550 3200 50  0000 C CNN
-F 2 "" V 9430 3000 50  0001 C CNN
+F 2 "Resistor_SMD:R_0603_1608Metric" V 9430 3000 50  0001 C CNN
 F 3 "~" H 9500 3000 50  0001 C CNN
 	1    9500 3000
@@
 F 0 "R40" V 9450 3250 50  0000 C CNN
 F 1 "0R0" V 9550 3650 50  0000 C CNN
-F 2 "" V 9430 3450 50  0001 C CNN
+F 2 "Resistor_SMD:R_0603_1608Metric" V 9430 3450 50  0001 C CNN
 F 3 "~" H 9500 3450 50  0001 C CNN
 	1    9500 3450
@@
 F 0 "R41" V 9450 3450 50  0000 C CNN
 F 1 "0R0" V 9550 3850 50  0000 C CNN
-F 2 "" V 9430 3650 50  0001 C CNN
+F 2 "Resistor_SMD:R_0603_1608Metric" V 9430 3650 50  0001 C CNN
 F 3 "~" H 9500 3650 50  0001 C CNN
 	1    9500 3650
@@
 F 0 "R37" H 9070 3296 50  0000 L CNN
 F 1 "0R0" H 9070 3205 50  0000 L CNN
-F 2 "" V 8930 3250 50  0001 C CNN
+F 2 "Resistor_SMD:R_0603_1608Metric" V 8930 3250 50  0001 C CNN
 F 3 "~" H 9000 3250 50  0001 C CNN
 	1    9000 3250
@@
 F 0 "R38" H 9070 3896 50  0000 L CNN
 F 1 "0R0" H 9070 3805 50  0000 L CNN
-F 2 "" V 8930 3850 50  0001 C CNN
+F 2 "Resistor_SMD:R_0603_1608Metric" V 8930 3850 50  0001 C CNN
 F 3 "~" H 9000 3850 50  0001 C CNN
 	1    9000 3850
@@
 F 0 "C48" V 7100 3200 50  0000 C CNN
 F 1 "1n" V 7200 3150 50  0000 C CNN
-F 2 "" H 7188 2900 50  0001 C CNN
+F 2 "Capacitor_SMD:C_0402_1005Metric" H 7188 2900 50  0001 C CNN
 F 3 "~" H 7150 3050 50  0001 C CNN
 	1    7150 3050
@@
 F 0 "C49" V 7100 3600 50  0000 C CNN
 F 1 "1n" V 7200 3550 50  0000 C CNN
-F 2 "" H 7188 3300 50  0001 C CNN
+F 2 "Capacitor_SMD:C_0402_1005Metric" H 7188 3300 50  0001 C CNN
 F 3 "~" H 7150 3450 50  0001 C CNN
 	1    7150 3450
@@
 F 0 "R35" H 6850 3300 50  0000 L CNN
 F 1 "52R3" H 6850 3200 50  0000 L CNN
-F 2 "" V 6730 3250 50  0001 C CNN
+F 2 "Resistor_SMD:R_0402_1005Metric" V 6730 3250 50  0001 C CNN
 F 3 "~" H 6800 3250 50  0001 C CNN
 	1    6800 3250
@@
 F 0 "U13" H 7750 3600 50  0000 C CNN
 F 1 "AD8302" H 7850 3500 50  0000 C CNN
-F 2 "" H 8550 3450 50  0001 L CNN
+F 2 "Package_SO:TSSOP-14_4.4x5mm_P0.65mm" H 8550 3450 50  0001 L CNN
 F 3 "" H 8550 3350 50  0001 L CNN
 	1    7500 3350
@@
 F 0 "C51" V 7200 4200 50  0000 C CNN
 F 1 "1n" V 7100 4150 50  0000 C CNN
-F 2 "" H 7188 3900 50  0001 C CNN
+F 2 "Capacitor_SMD:C_0402_1005Metric" H 7188 3900 50  0001 C CNN
 F 3 "~" H 7150 4050 50  0001 C CNN
 	1    7150 4050
@@
 F 0 "C50" V 7200 3800 50  0000 C CNN
 F 1 "1n" V 7100 3750 50  0000 C CNN
-F 2 "" H 7188 3500 50  0001 C CNN
+F 2 "Capacitor_SMD:C_0402_1005Metric" H 7188 3500 50  0001 C CNN
 F 3 "~" H 7150 3650 50  0001 C CNN
 	1    7150 3650
@@
 F 0 "R36" H 6850 3800 50  0000 L CNN
 F 1 "52R3" H 6850 3900 50  0000 L CNN
-F 2 "" V 6730 3850 50  0001 C CNN
+F 2 "Resistor_SMD:R_0402_1005Metric" V 6730 3850 50  0001 C CNN
 F 3 "~" H 6800 3850 50  0001 C CNN
 	1    6800 3850
@@
 $EndComp
 $Comp
-L power:GND #PWR0112
+L power:GND #PWR070
 U 1 1 5CF3E890
 P 6600 3600
-F 0 "#PWR0112" H 6600 3350 50  0001 C CNN
+F 0 "#PWR070" H 6600 3350 50  0001 C CNN
 F 1 "GND" H 6605 3427 50  0000 C CNN
 F 2 "" H 6600 3600 50  0001 C CNN
@@
 $EndComp
 $Comp
-L power:GND #PWR0113
+L power:GND #PWR073
 U 1 1 5CF90B48
 P 8500 2900
-F 0 "#PWR0113" H 8500 2650 50  0001 C CNN
+F 0 "#PWR073" H 8500 2650 50  0001 C CNN
 F 1 "GND" H 8505 2727 50  0000 C CNN
 F 2 "" H 8500 2900 50  0001 C CNN
@@
 F 0 "R33" H 2770 4296 50  0000 L CNN
 F 1 "150R" H 2770 4205 50  0000 L CNN
-F 2 "" V 2630 4250 50  0001 C CNN
+F 2 "Resistor_SMD:R_0402_1005Metric" V 2630 4250 50  0001 C CNN
 F 3 "~" H 2700 4250 50  0001 C CNN
 	1    2700 4250

Commit message: prelim schematic capture complete
Parts:
- renumbered C47 to C49, C48 to C50, C49 to C51, C50 to C52, C51 to C53, C52 to C54, C53 to C55, C54 to C56, C55 to C57, R26 to R33, R27 to R34, R28 to R35, R29 to R36, R30 to R37, R31 to R38, R32 to R39, R33 to R40, R34 to R41, R35 to R42, R36 to R43, R37 to R44, R38 to R45, R39 to R46, R40 to R47, R41 to R48, U12 to U14, U13 to U15

Commit message: all 3d models created, prelim bom generated
Parts:
- added D16, D17: LED, LED_SMD:LED_0603_1608Metric, symbol Device:LED
- added R59, R60: 470R, Resistor_SMD:R_0603_1608Metric, symbol Device:R
- added TP17, TP18, TP19: TP, TestPoint:TestPoint_Pad_D1.0mm, symbol Connector:TestPoint
Connections:
- wire segments 120 -> 137
Other:
- moved on the sheet: C49, C55, C56, R33, R34, R35, R36, R37, R38, R39, R40, R41

Commit message: More schematic changes + updated functionals
Parts:
- removed U14: PE4257, VNA_Footprints:QFN-20-1EP_4x4mm_P0.5mm_EP2.15x2.15mm_ThermalVias, symbol VNA_Symbols:PE4257
- added U14: F2923, VNA_Footprints:QFN-20-1EP_4x4mm_P0.5mm_EP2x2mm_ThermalVias, symbol VNA_Symbols:F2923
Other:
- note added: "Sets two \nwire ctrl"
- moved on the sheet: C49, C50, C51, C52, C53, C54, C55, C56, C57, D16, D17, R33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

Commit message: first day of layout / routing done
Connections:
- net at R38.1, R41.1: now also U14.3 (RF1); no longer U14.13 (RF2)
- net at R37.1, R40.1: now also U14.13 (RF2); no longer U14.3 (RF1)
Other:
- moved on the sheet: R34, R35, R37, R38, R40, R41
Changed lines of the file:
@@
 Comment4 ""
 $EndDescr
-Text HLabel 1550 5000 0    50   Input ~ 6
+Text HLabel 1550 4000 0    50   Input ~ 10
 RF_THROUGH
+Wire Wire Line
+	1900 5000 1800 5000
+Wire Wire Line
+	1800 5000 1800 5100
+Wire Wire Line
+	2200 5000 2300 5000
+Wire Wire Line
+	2300 5000 2300 5100
+Wire Wire Line
+	1800 5400 1800 5450
+Wire Wire Line
+	2300 5400 2300 5450
+Wire Wire Line
+	1800 5000 1550 5000
+Connection ~ 1800 5000
+Text HLabel 1550 5000 0    50   Input ~ 10
+RF_REVERSE
 Wire Wire Line
 	1900 4000 1800 4000
@@
 	1800 4000 1550 4000
 Connection ~ 1800 4000
-Text HLabel 1550 4000 0    50   Input ~ 6
-RF_REVERSE
-Wire Wire Line
-	1900 5000 1800 5000
-Wire Wire Line
-	1800 5000 1800 5100
-Wire Wire Line
-	2200 5000 2300 5000
-Wire Wire Line
-	2300 5000 2300 5100
-Wire Wire Line
-	1800 5400 1800 5450
-Wire Wire Line
-	2300 5400 2300 5450
-Wire Wire Line
-	1800 5000 1550 5000
-Connection ~ 1800 5000
-Text Notes 1900 5450 0    50   ~ 6
+Text Notes 1900 4450 0    50   ~ 10
 -21 dB
+Wire Wire Line
+	4150 4150 2700 4150
 Connection ~ 2300 4000
-Wire Wire Line
-	4150 4150 2800 4150
-Connection ~ 2300 5000
-Text HLabel 3150 4350 0    50   Input ~ 6
+Text HLabel 3150 4350 0    50   Input ~ 10
 CTRL_1
-Text HLabel 3150 4450 0    50   Input ~ 6
+Text HLabel 3150 4450 0    50   Input ~ 10
 CTRL_2
 Wire Wire Line
@@
 	5600 5150 5600 5100
 Connection ~ 5600 5100
-Text HLabel 1550 3000 0    50   Input ~ 6
+Text HLabel 1550 3000 0    50   Input ~ 10
 RF_FORWARD
 Wire Wire Line
@@
 	4900 3350 4900 3500
 Connection ~ 4900 3500
-Text HLabel 9800 2950 2    50   Output ~ 6
+Text HLabel 9800 2950 2    50   Output ~ 10
 VMAG
-Text HLabel 9800 3400 2    50   Output ~ 6
+Text HLabel 9800 3400 2    50   Output ~ 10
 VREF
-Text HLabel 9800 3600 2    50   Output ~ 6
+Text HLabel 9800 3600 2    50   Output ~ 10
 VPHS
-Text HLabel 4900 3350 1    50   Input ~ 6
+Text HLabel 4900 3350 1    50   Input ~ 10
 3V3A
 Wire Wire Line
@@
 Wire Wire Line
 	2300 3000 6800 3000
-Text HLabel 8100 2200 1    50   Input ~ 6
+Text HLabel 8100 2200 1    50   Input ~ 10
 3V3A
 Wire Wire Line
@@
 Wire Wire Line
 	8550 2700 8550 2850
-Text Notes 4250 2800 0    100  ~ 6
+Text Notes 4250 2800 0    100  ~ 20
 Path Select
-Text Notes 7400 1800 0    100  ~ 6
+Text Notes 7400 1800 0    100  ~ 20
 AD8302 Gain Phase Detector
-Text Notes 1900 4500 0    50   ~ 6
+Text Notes 1900 5500 0    50   ~ 10
 -6 dB
 $Comp
 L Device:R R37
 U 1 1 5CD9F648
+P 2050 5000
+F 0 "R37" V 1950 5000 50  0000 C CNN
+F 1 "37R" V 2150 5000 50  0000 C CNN
+F 2 "Resistor_SMD:R_0402_1005Metric" V 1980 5000 50  0001 C CNN
+F 3 "~" H 2050 5000 50  0001 C CNN
+	1    2050 5000
+	0    1    1    0
+$EndComp
+$Comp
+L Device:R R34
+U 1 1 5CDA074A
+P 1800 5250
+F 0 "R34" H 1870 5296 50  0000 L CNN
+F 1 "150R" H 1870 5205 50  0000 L CNN
+F 2 "Resistor_SMD:R_0402_1005Metric" V 1730 5250 50  0001 C CNN
+F 3 "~" H 1800 5250 50  0001 C CNN
+	1    1800 5250
+	1    0    0    -1
+$EndComp
+$Comp
+L power:GND #PWR087
+U 1 1 5CDA106C
+P 2300 5450
+F 0 "#PWR087" H 2300 5200 50  0001 C CNN
+F 1 "GND" H 2305 5277 50  0000 C CNN
+F 2 "" H 2300 5450 50  0001 C CNN
+F 3 "" H 2300 5450 50  0001 C CNN
+	1    2300 5450
+	1    0    0    -1
+$EndComp
+$Comp
+L power:GND #PWR084
+U 1 1 5CDA1618
+P 1800 5450
+F 0 "#PWR084" H 1800 5200 50  0001 C CNN
+F 1 "GND" H 1805 5277 50  0000 C CNN
+F 2 "" H 1800 5450 50  0001 C CNN
+F 3 "" H 1800 5450 50  0001 C CNN
+	1    1800 5450
+	1    0    0    -1
+$EndComp
+$Comp
+L Device:R R38
+U 1 1 5CDA4337
 P 2050 4000
-F 0 "R37" V 1950 4000 50  0000 C CNN
-F 1 "37R" V 2150 4000 50  0000 C CNN
+F 0 "R38" V 1950 4000 50  0000 C CNN
+F 1 "278R" V 2150 4000 50  0000 C CNN
 F 2 "Resistor_SMD:R_0402_1005Metric" V 1980 4000 50  0001 C CNN
 F 3 "~" H 2050 4000 50  0001 C CNN
@@
 $EndComp
 $Comp
-L Device:R R34
-U 1 1 5CDA074A
-P 1800 4250
-F 0 "R34" H 1870 4296 50  0000 L CNN
-F 1 "150R" H 1870 4205 50  0000 L CNN
-F 2 "Resistor_SMD:R_0402_1005Metric" V 1730 4250 50  0001 C CNN
-F 3 "~" H 1800 4250 50  0001 C CNN
-	1    1800 4250
-	1    0    0    -1
-$EndComp
-$Comp
-L power:GND #PWR087
-U 1 1 5CDA106C
+L Device:R R41
+U 1 1 5CDA433D
+P 2300 4250
+F 0 "R41" H 2370 4296 50  0000 L CNN
+F 1 "60R" H 2370 4205 50  0000 L CNN
+F 2 "Resistor_SMD:R_0402_1005Metric" V 2230 4250 50  0001 C CNN
+F 3 "~" H 2300 4250 50  0001 C CNN
+	1    2300 4250
+	1    0    0    -1
+$EndComp
+$Comp
+L power:GND #PWR088
+U 1 1 5CDA434F
 P 2300 4450
-F 0 "#PWR087" H 2300 4200 50  0001 C CNN
+F 0 "#PWR088" H 2300 4200 50  0001 C CNN
 F 1 "GND" H 2305 4277 50  0000 C CNN
 F 2 "" H 2300 4450 50  0001 C CNN
@@
 $EndComp
 $Comp
-L power:GND #PWR084
-U 1 1 5CDA1618
+L power:GND #PWR085
+U 1 1 5CDA4355
 P 1800 4450
-F 0 "#PWR084" H 1800 4200 50  0001 C CNN
+F 0 "#PWR085" H 1800 4200 50  0001 C CNN
 F 1 "GND" H 1805 4277 50  0000 C CNN
 F 2 "" H 1800 4450 50  0001 C CNN
@@
 $EndComp
 $Comp
-L Device:R R38
-U 1 1 5CDA4337
-P 2050 5000
-F 0 "R38" V 1950 5000 50  0000 C CNN
-F 1 "278R" V 2150 5000 50  0000 C CNN
-F 2 "Resistor_SMD:R_0402_1005Metric" V 1980 5000 50  0001 C CNN
-F 3 "~" H 2050 5000 50  0001 C CNN
-	1    2050 5000
-	0    1    1    0
-$EndComp
-$Comp
-L Device:R R41
-U 1 1 5CDA433D
-P 2300 5250
-F 0 "R41" H 2370 5296 50  0000 L CNN
-F 1 "60R" H 2370 5205 50  0000 L CNN
-F 2 "Resistor_SMD:R_0402_1005Metric" V 2230 5250 50  0001 C CNN
-F 3 "~" H 2300 5250 50  0001 C CNN
-	1    2300 5250
-	1    0    0    -1
-$EndComp
-$Comp
-L power:GND #PWR088
-U 1 1 5CDA434F
-P 2300 5450
-F 0 "#PWR088" H 2300 5200 50  0001 C CNN
-F 1 "GND" H 2305 5277 50  0000 C CNN
-F 2 "" H 2300 5450 50  0001 C CNN
-F 3 "" H 2300 5450 50  0001 C CNN
-	1    2300 5450
-	1    0    0    -1
-$EndComp
-$Comp
-L power:GND #PWR085
-U 1 1 5CDA4355
-P 1800 5450
-F 0 "#PWR085" H 1800 5200 50  0001 C CNN
-F 1 "GND" H 1805 5277 50  0000 C CNN
-F 2 "" H 1800 5450 50  0001 C CNN
-F 3 "" H 1800 5450 50  0001 C CNN
-	1    1800 5450
-	1    0    0    -1
-$EndComp
-$Comp
 L Device:R R35
 U 1 1 5CDA469F
-P 1800 5250
-F 0 "R35" H 1870 5296 50  0000 L CNN
-F 1 "60R" H 1870 5205 50  0000 L CNN
-F 2 "Resistor_SMD:R_0402_1005Metric" V 1730 5250 50  0001 C CNN
-F 3 "~" H 1800 5250 50  0001 C CNN
-	1    1800 5250
+P 1800 4250
+F 0 "R35" H 1870 4296 50  0000 L CNN
+F 1 "60R" H 1870 4205 50  0000 L CNN
+F 2 "Resistor_SMD:R_0402_1005Metric" V 1730 4250 50  0001 C CNN
+F 3 "~" H 1800 4250 50  0001 C CNN
+	1    1800 4250
 	1    0    0    -1
 $EndComp
@@
 L Device:R R40
 U 1 1 5CFA7BB2
-P 2300 4250
-F 0 "R40" H 2370 4296 50  0000 L CNN
-F 1 "150R" H 2370 4205 50  0000 L CNN
-F 2 "Resistor_SMD:R_0402_1005Metric" V 2230 4250 50  0001 C CNN
-F 3 "~" H 2300 4250 50  0001 C CNN
-	1    2300 4250
+P 2300 5250
+F 0 "R40" H 2370 5296 50  0000 L CNN
+F 1 "150R" H 2370 5205 50  0000 L CNN
+F 2 "Resistor_SMD:R_0402_1005Metric" V 2230 5250 50  0001 C CNN
+F 3 "~" H 2300 5250 50  0001 C CNN
+	1    2300 5250
 	1    0    0    -1
 $EndComp
@@
 $EndComp
 Wire Wire Line
-	2800 4150 2800 5000
-Wire Wire Line
-	2300 5000 2800 5000
-Wire Wire Line
-	2300 4000 4150 4000
+	2700 4150 2700 5000
 Connection ~ 3200 4350
 Connection ~ 3600 4450
@@
 	5750 4000 6800 4000
 Connection ~ 2300 3000
-Text Notes 3900 5100 0    50   ~ 6
+Text Notes 3900 5100 0    50   ~ 10
 Sets two \nwire ctrl
 Wire Wire Line
 	4900 3500 4900 3800
+Wire Wire Line
+	2300 4000 4150 4000
+Wire Wire Line
+	2700 5000 2300 5000
+Connection ~ 2300 5000
 $EndSCHEMATC
