File: Hardware/VNA/power.sch (KiCad schematic (older format))
At the start: 13 parts, among them U2 TVL755P, U3 LP5912, U4 MIC5366-1.8

Commit message: added footprints and 3d models
Parts:
- C28, C29, C30, C31: footprint (none) -> Capacitor_SMD:C_0603_1608Metric
- C32, C33: footprint Capacitor_SMD:C_0402_1005Metric -> Capacitor_SMD:C_0603_1608Metric
- F1: footprint (none) -> Fuse:Fuse_1206_3216Metric
- U2, U3: footprint (none) -> Package_DFN_QFN:DFN-6-1EP_2x2mm_P0.65mm_EP1x1.6mm
- U4: footprint (none) -> Package_TO_SOT_SMD:SOT-353_SC-70-5
Changed lines of the file:
@@
 F 0 "C32" H 8415 3546 50  0000 L CNN
 F 1 "1u" H 8415 3455 50  0000 L CNN
-F 2 "Capacitor_SMD:C_0402_1005Metric" H 8338 3350 50  0001 C CNN
+F 2 "Capacitor_SMD:C_0603_1608Metric" H 8338 3350 50  0001 C CNN
 F 3 "~" H 8300 3500 50  0001 C CNN
 	1    8300 3500
@@
 F 0 "C33" H 9915 3546 50  0000 L CNN
 F 1 "1u" H 9915 3455 50  0000 L CNN
-F 2 "Capacitor_SMD:C_0402_1005Metric" H 9838 3350 50  0001 C CNN
+F 2 "Capacitor_SMD:C_0603_1608Metric" H 9838 3350 50  0001 C CNN
 F 3 "~" H 9800 3500 50  0001 C CNN
 	1    9800 3500
@@
 F 0 "U4" H 9225 3765 50  0000 C CNN
 F 1 "MIC5366-1.8" H 9225 3674 50  0000 C CNN
-F 2 "" H 9000 3700 50  0001 C CNN
+F 2 "Package_TO_SOT_SMD:SOT-353_SC-70-5" H 9000 3700 50  0001 C CNN
 F 3 "" H 9000 3700 50  0001 C CNN
 	1    9200 3400
@@
 F 0 "C30" H 6265 3546 50  0000 L CNN
 F 1 "1u" H 6265 3455 50  0000 L CNN
-F 2 "" H 6188 3350 50  0001 C CNN
+F 2 "Capacitor_SMD:C_0603_1608Metric" H 6188 3350 50  0001 C CNN
 F 3 "~" H 6150 3500 50  0001 C CNN
 	1    6150 3500
@@
 F 0 "U3" H 6650 4000 49  0000 C CNN
 F 1 "LP5912" H 6750 3900 49  0000 C CNN
-F 2 "" H 6750 3900 49  0001 C CNN
+F 2 "Package_DFN_QFN:DFN-6-1EP_2x2mm_P0.65mm_EP1x1.6mm" H 6750 3900 49  0001 C CNN
 F 3 "" H 6750 3900 49  0001 C CNN
 	1    6800 3550
@@
 F 0 "C31" H 7615 3546 50  0000 L CNN
 F 1 "1u" H 7615 3455 50  0000 L CNN
-F 2 "" H 7538 3350 50  0001 C CNN
+F 2 "Capacitor_SMD:C_0603_1608Metric" H 7538 3350 50  0001 C CNN
 F 3 "~" H 7500 3500 50  0001 C CNN
 	1    7500 3500
@@
 F 0 "U2" H 4525 3875 50  0000 C CNN
 F 1 "TVL755P" H 4525 3784 50  0000 C CNN
-F 2 "" H 4500 3900 100 0001 C CNN
+F 2 "Package_DFN_QFN:DFN-6-1EP_2x2mm_P0.65mm_EP1x1.6mm" H 4500 3900 100 0001 C CNN
 F 3 "" H 4500 3900 100 0001 C CNN
 	1    4500 3450
@@
 F 0 "C28" H 3865 3496 50  0000 L CNN
 F 1 "1u" H 3865 3405 50  0000 L CNN
-F 2 "" H 3788 3300 50  0001 C CNN
+F 2 "Capacitor_SMD:C_0603_1608Metric" H 3788 3300 50  0001 C CNN
 F 3 "~" H 3750 3450 50  0001 C CNN
 	1    3750 3450
@@
 F 0 "C29" H 5365 3496 50  0000 L CNN
 F 1 "1u" H 5365 3405 50  0000 L CNN
-F 2 "" H 5288 3300 50  0001 C CNN
+F 2 "Capacitor_SMD:C_0603_1608Metric" H 5288 3300 50  0001 C CNN
 F 3 "~" H 5250 3450 50  0001 C CNN
 	1    5250 3450
@@
 F 0 "F1" V 2000 2100 50  0000 C CNN
 F 1 "500mA Polyfuse" V 2200 2100 50  0000 C CNN
-F 2 "" H 2150 1900 50  0001 L CNN
+F 2 "Fuse:Fuse_1206_3216Metric" H 2150 1900 50  0001 L CNN
 F 3 "~" H 2100 2100 50  0001 C CNN
 	1    2100 2100
@@
 	1550 2100 2000 2100
 $Comp
-L power:PWR_FLAG #FLG0101
+L power:PWR_FLAG #FLG01
 U 1 1 5CAD0E34
 P 2600 2200
-F 0 "#FLG0101" H 2600 2275 50  0001 C CNN
+F 0 "#FLG01" H 2600 2275 50  0001 C CNN
 F 1 "PWR_FLAG" V 2600 2328 50  0000 L CNN
 F 2 "" H 2600 2200 50  0001 C CNN
@@
 	2500 2200 2600 2200
 $Comp
-L power:PWR_FLAG #FLG0102
+L power:PWR_FLAG #FLG02
 U 1 1 5CADABE9
 P 3150 3250
-F 0 "#FLG0102" H 3150 3325 50  0001 C CNN
+F 0 "#FLG02" H 3150 3325 50  0001 C CNN
 F 1 "PWR_FLAG" V 3150 3378 50  0000 L CNN
 F 2 "" H 3150 3250 50  0001 C CNN

Commit message: prelim schematic capture complete
Parts:
- removed FB3: BLM18PG181SN1D, VNA_Footprints:BEADC1608X95N, symbol Device:Ferrite_Bead
- added D2, D3, D4, D5, D6: LED, symbol Device:LED
- added FB4: Bead, symbol VNA_Symbols:Ferrite_Bead_PWR
- added Q1: RE1C002UN, symbol Device:Q_NMOS_GSD
- added R13: 10K, symbol Device:R
- added R14, R15, R16: 470R, symbol Device:R
- added R17, R18: 1K, symbol Device:R
- added TP1: VBUS, symbol Connector:TestPoint
- added TP10, TP11, TP12, TP13, TP14, TP15, TP6, TP7, TP8, TP9: GND, symbol Connector:TestPoint
- added TP2: 5V0, symbol Connector:TestPoint
- added TP3: 3V3A, symbol Connector:TestPoint
- added TP4: 1V8, symbol Connector:TestPoint
- added TP5: 3V3, symbol Connector:TestPoint
- renumbered C30 to C28, C26 to C29, C27 to C30, C28 to C32, C32 to C33, C29 to C34, C33 to C35, U3 to U4, U2 to U5, U4 to U6
Connections:
- wire segments 72 -> 105
Other:
- note added: "Ground Test Points"
- note added: "Voltage Rail LEDs"
- moved on the sheet: C28, C29, C30, C31, C32, C33, C34, C35, F1, U4, U6

Commit message: all 3d models created, prelim bom generated
Parts:
- D2, D3, D4, D5, D6: footprint (none) -> LED_SMD:LED_0603_1608Metric
- F1: footprint Fuse:Fuse_1206_3216Metric -> VNA_Footprints:Fuse_1206_3216Metric
- FB4: footprint (none) -> VNA_Footprints:BEADC1608X95N
- Q1: footprint (none) -> Package_TO_SOT_SMD:SOT-89-3
- R13, R14, R15, R16, R17, R18: footprint (none) -> Resistor_SMD:R_0603_1608Metric
- TP1, TP10, TP2, TP3, TP4, TP5, TP6, TP7, TP8, TP9: footprint (none) -> TestPoint:TestPoint_Pad_D1.0mm
- TP11, TP12, TP13, TP14, TP15: footprint (none) -> VNA_Footprints:S1751-46_smdTestPoint
Changed lines of the file:
@@
 	5150 3950 5150 3800
 Connection ~ 4950 3950
-Text Notes 4000 3550 0    100  ~ 6
+Text Notes 4000 3550 0    100  ~ 0
 1V8 LDO\n
 Wire Wire Line
@@
 	1    0    0    -1
 $EndComp
-Text Notes 1300 2150 0    100  ~ 6
+Text Notes 1300 2150 0    100  ~ 0
 5V (Filtered)
-Text HLabel 3350 3800 1    49   Input ~ 6
+Text HLabel 3350 3800 1    49   Input ~ 0
 3V3A
-Text HLabel 5150 3800 1    49   Input ~ 6
+Text HLabel 5150 3800 1    49   Input ~ 0
 1V8
-Text HLabel 2550 2400 1    49   Input ~ 6
+Text HLabel 2550 2400 1    49   Input ~ 0
 5V0
 Wire Wire Line
@@
 	1    0    0    -1
 $EndComp
-Text Notes 2250 3600 2    100  ~ 6
+Text Notes 2250 3600 2    100  ~ 0
 3V3A LDO
 Wire Wire Line
@@
 Wire Wire Line
 	2550 3950 2850 3950
-Text HLabel 2850 3850 1    49   Input ~ 6
+Text HLabel 2850 3850 1    49   Input ~ 0
 3V3A
 Connection ~ 2550 3950
@@
 Wire Wire Line
 	4950 2500 5250 2500
-Text HLabel 5250 2400 1    49   Input ~ 6
+Text HLabel 5250 2400 1    49   Input ~ 0
 3V3
 Connection ~ 4950 2500
@@
 $EndComp
 Connection ~ 3750 2500
-Text Notes 4600 2200 2    100  ~ 6
+Text Notes 4600 2200 2    100  ~ 0
 3V3 LDO
 $Comp
@@
 F 0 "F1" V 1700 1400 50  0000 C CNN
 F 1 "500mA Polyfuse" V 1900 1400 50  0000 C CNN
-F 2 "Fuse:Fuse_1206_3216Metric" H 1850 1200 50  0001 L CNN
+F 2 "VNA_Footprints:Fuse_1206_3216Metric" H 1850 1200 50  0001 L CNN
 F 3 "~" H 1800 1400 50  0001 C CNN
 	1    1800 1400
 	0    1    1    0
 $EndComp
-Text HLabel 1250 1400 0    49   Input ~ 6
+Text HLabel 1250 1400 0    49   Input ~ 0
 VBUS
 Wire Wire Line
 	1900 1400 2200 1400
-Text Label 2300 1400 0    50   ~ 6
+Text Label 2300 1400 0    50   ~ 0
 VIN
-Text Label 1050 2400 1    50   ~ 6
+Text Label 1050 2400 1    50   ~ 0
 VIN
-Text Label 3350 2400 1    50   ~ 6
+Text Label 3350 2400 1    50   ~ 0
 VIN
-Text Label 1100 3850 1    50   ~ 6
+Text Label 1100 3850 1    50   ~ 0
 VIN
-Text Notes 1200 1150 0    100  ~ 6
+Text Notes 1200 1150 0    100  ~ 0
 Input Protection
 Wire Wire Line
@@
 F 0 "TP4" V 5075 4250 50  0000 R CNN
 F 1 "1V8" V 5150 4250 50  0000 R CNN
-F 2 "" H 5350 3950 50  0001 C CNN
+F 2 "TestPoint:TestPoint_Pad_D1.0mm" H 5350 3950 50  0001 C CNN
 F 3 "~" H 5350 3950 50  0001 C CNN
 	1    5150 3950
@@
 F 0 "Q1" H 6706 3546 50  0000 L CNN
 F 1 "RE1C002UN" H 6706 3455 50  0000 L CNN
-F 2 "" H 6700 3600 50  0001 C CNN
+F 2 "Package_TO_SOT_SMD:SOT-89-3" H 6700 3600 50  0001 C CNN
 F 3 "~" H 6500 3500 50  0001 C CNN
 	1    6500 3500
@@
 F 0 "R13" V 6475 3750 50  0000 L CNN
 F 1 "10K" V 6400 3675 50  0000 L CNN
-F 2 "" V 6330 3750 50  0001 C CNN
+F 2 "Resistor_SMD:R_0603_1608Metric" V 6330 3750 50  0001 C CNN
 F 3 "~" H 6400 3750 50  0001 C CNN
 	1    6400 3750
@@
 Wire Wire Line
 	6600 2600 6600 2550
-Text HLabel 6600 2550 1    50   Input ~ 6
+Text HLabel 6600 2550 1    50   Input ~ 0
 3V3A
-Text HLabel 6150 3500 0    50   Input ~ 6
+Text HLabel 6150 3500 0    50   Input ~ 0
 1V8
 Wire Wire Line
@@
 F 0 "D2" V 6639 2983 50  0000 R CNN
 F 1 "LED" V 6548 2983 50  0000 R CNN
-F 2 "" H 6600 3100 50  0001 C CNN
+F 2 "LED_SMD:LED_0603_1608Metric" H 6600 3100 50  0001 C CNN
 F 3 "~" H 6600 3100 50  0001 C CNN
 	1    6600 3100
@@
 F 0 "R14" H 6670 2796 50  0000 L CNN
 F 1 "470R" H 6670 2705 50  0000 L CNN
-F 2 "" V 6530 2750 50  0001 C CNN
+F 2 "Resistor_SMD:R_0603_1608Metric" V 6530 2750 50  0001 C CNN
 F 3 "~" H 6600 2750 50  0001 C CNN
 	1    6600 2750
 	1    0    0    -1
 $EndComp
-Text Notes 6800 2200 0    100  ~ 6
+Text Notes 6800 2200 0    100  ~ 0
 Voltage Rail LEDs
 Wire Wire Line
 	7250 2600 7250 2550
-Text HLabel 7250 2550 1    50   Input ~ 6
+Text HLabel 7250 2550 1    50   Input ~ 0
 3V3A
 Wire Wire Line
@@
 F 0 "D3" V 7289 2983 50  0000 R CNN
 F 1 "LED" V 7198 2983 50  0000 R CNN
-F 2 "" H 7250 3100 50  0001 C CNN
+F 2 "LED_SMD:LED_0603_1608Metric" H 7250 3100 50  0001 C CNN
 F 3 "~" H 7250 3100 50  0001 C CNN
 	1    7250 3100
@@
 F 0 "R15" H 7320 2796 50  0000 L CNN
 F 1 "470R" H 7320 2705 50  0000 L CNN
-F 2 "" V 7180 2750 50  0001 C CNN
+F 2 "Resistor_SMD:R_0603_1608Metric" V 7180 2750 50  0001 C CNN
 F 3 "~" H 7250 2750 50  0001 C CNN
 	1    7250 2750
@@
 Wire Wire Line
 	7650 2600 7650 2550
-Text HLabel 7650 2550 1    50   Input ~ 6
+Text HLabel 7650 2550 1    50   Input ~ 0
 3V3
 Wire Wire Line
@@
 F 0 "D4" V 7689 2983 50  0000 R CNN
 F 1 "LED" V 7598 2983 50  0000 R CNN
-F 2 "" H 7650 3100 50  0001 C CNN
+F 2 "LED_SMD:LED_0603_1608Metric" H 7650 3100 50  0001 C CNN
 F 3 "~" H 7650 3100 50  0001 C CNN
 	1    7650 3100
@@
 F 0 "R16" H 7720 2796 50  0000 L CNN
 F 1 "470R" H 7720 2705 50  0000 L CNN
-F 2 "" V 7580 2750 50  0001 C CNN
+F 2 "Resistor_SMD:R_0603_1608Metric" V 7580 2750 50  0001 C CNN
 F 3 "~" H 7650 2750 50  0001 C CNN
 	1    7650 2750
@@
 Wire Wire Line
 	8050 2600 8050 2550
-Text HLabel 8050 2550 1    50   Input ~ 6
+Text HLabel 8050 2550 1    50   Input ~ 0
 5V0
 Wire Wire Line
@@
 F 0 "D5" V 8089 2983 50  0000 R CNN
 F 1 "LED" V 7998 2983 50  0000 R CNN
-F 2 "" H 8050 3100 50  0001 C CNN
+F 2 "LED_SMD:LED_0603_1608Metric" H 8050 3100 50  0001 C CNN
 F 3 "~" H 8050 3100 50  0001 C CNN
 	1    8050 3100
@@
 F 0 "R17" H 8120 2796 50  0000 L CNN
 F 1 "1K" H 8120 2705 50  0000 L CNN
-F 2 "" V 7980 2750 50  0001 C CNN
+F 2 "Resistor_SMD:R_0603_1608Metric" V 7980 2750 50  0001 C CNN
 F 3 "~" H 8050 2750 50  0001 C CNN
 	1    8050 2750
@@
 F 0 "D6" V 8439 2983 50  0000 R CNN
 F 1 "LED" V 8348 2983 50  0000 R CNN
-F 2 "" H 8400 3100 50  0001 C CNN
+F 2 "LED_SMD:LED_0603_1608Metric" H 8400 3100 50  0001 C CNN
 F 3 "~" H 8400 3100 50  0001 C CNN
 	1    8400 3100
@@
 F 0 "R18" H 8470 2796 50  0000 L CNN
 F 1 "1K" H 8470 2705 50  0000 L CNN
-F 2 "" V 8330 2750 50  0001 C CNN
+F 2 "Resistor_SMD:R_0603_1608Metric" V 8330 2750 50  0001 C CNN
 F 3 "~" H 8400 2750 50  0001 C CNN
 	1    8400 2750
@@
 	1    0    0    -1
 $EndComp
-Text HLabel 8400 2550 1    49   Input ~ 6
+Text HLabel 8400 2550 1    49   Input ~ 0
 VBUS
 Connection ~ 5150 3950
@@
 F 0 "TP5" V 5175 2800 50  0000 R CNN
 F 1 "3V3" V 5250 2800 50  0000 R CNN
-F 2 "" H 5450 2500 50  0001 C CNN
+F 2 "TestPoint:TestPoint_Pad_D1.0mm" H 5450 2500 50  0001 C CNN
 F 3 "~" H 5450 2500 50  0001 C CNN
 	1    5250 2500
@@
 F 0 "TP3" V 2775 4250 50  0000 R CNN
 F 1 "3V3A" V 2850 4300 50  0000 R CNN
-F 2 "" H 3050 3950 50  0001 C CNN
+F 2 "TestPoint:TestPoint_Pad_D1.0mm" H 3050 3950 50  0001 C CNN
 F 3 "~" H 3050 3950 50  0001 C CNN
 	1    2850 3950
@@
 F 0 "TP2" V 2675 2850 50  0000 R CNN
 F 1 "5V0" V 2750 2850 50  0000 R CNN
-F 2 "" H 2950 2550 50  0001 C CNN
+F 2 "TestPoint:TestPoint_Pad_D1.0mm" H 2950 2550 50  0001 C CNN
 F 3 "~" H 2950 2550 50  0001 C CNN
 	1    2750 2550
@@
 F 0 "TP1" H 1425 1675 50  0000 R CNN
 F 1 "VBUS" H 1425 1750 50  0000 R CNN
-F 2 "" H 1550 1450 50  0001 C CNN
+F 2 "TestPoint:TestPoint_Pad_D1.0mm" H 1550 1450 50  0001 C CNN
 F 3 "~" H 1550 1450 50  0001 C CNN
 	1    1350 1450
@@
 F 0 "TP7" H 9258 3068 50  0000 L CNN
 F 1 "GND" H 9258 2977 50  0000 L CNN
-F 2 "" H 9400 2950 50  0001 C CNN
+F 2 "TestPoint:TestPoint_Pad_D1.0mm" H 9400 2950 50  0001 C CNN
 F 3 "~" H 9400 2950 50  0001 C CNN
 	1    9200 2950
@@
 F 0 "TP9" H 9608 3068 50  0000 L CNN
 F 1 "GND" H 9608 2977 50  0000 L CNN
-F 2 "" H 9750 2950 50  0001 C CNN
+F 2 "TestPoint:TestPoint_Pad_D1.0mm" H 9750 2950 50  0001 C CNN
 F 3 "~" H 9750 2950 50  0001 C CNN
 	1    9550 2950
@@
 F 0 "TP11" H 9958 3068 50  0000 L CNN
 F 1 "GND" H 9958 2977 50  0000 L CNN
-F 2 "" H 10100 2950 50  0001 C CNN
+F 2 "VNA_Footprints:S1751-46_smdTestPoint" H 10100 2950 50  0001 C CNN
 F 3 "~" H 10100 2950 50  0001 C CNN
 	1    9900 2950
@@
 F 0 "TP13" H 10308 3068 50  0000 L CNN
 F 1 "GND" H 10308 2977 50  0000 L CNN
-F 2 "" H 10450 2950 50  0001 C CNN
+F 2 "VNA_Footprints:S1751-46_smdTestPoint" H 10450 2950 50  0001 C CNN
 F 3 "~" H 10450 2950 50  0001 C CNN
 	1    10250 2950
@@
 F 0 "TP15" H 10608 3068 50  0000 L CNN
 F 1 "GND" H 10608 2977 50  0000 L CNN
-F 2 "" H 10750 2950 50  0001 C CNN
+F 2 "VNA_Footprints:S1751-46_smdTestPoint" H 10750 2950 50  0001 C CNN
 F 3 "~" H 10750 2950 50  0001 C CNN
 	1    10550 2950
@@
 	1    0    0    -1
 $EndComp
-Text Notes 9150 2200 0    100  ~ 6
+Text Notes 9150 2200 0    100  ~ 0
 Ground Test Points
 $Comp
@@
 F 0 "TP6" H 9258 2568 50  0000 L CNN
 F 1 "GND" H 9258 2477 50  0000 L CNN
-F 2 "" H 9400 2450 50  0001 C CNN
+F 2 "TestPoint:TestPoint_Pad_D1.0mm" H 9400 2450 50  0001 C CNN
 F 3 "~" H 9400 2450 50  0001 C CNN
 	1    9200 2450
@@
 F 0 "TP8" H 9608 2568 50  0000 L CNN
 F 1 "GND" H 9608 2477 50  0000 L CNN
-F 2 "" H 9750 2450 50  0001 C CNN
+F 2 "TestPoint:TestPoint_Pad_D1.0mm" H 9750 2450 50  0001 C CNN
 F 3 "~" H 9750 2450 50  0001 C CNN
 	1    9550 2450
@@
 F 0 "TP10" H 9958 2568 50  0000 L CNN
 F 1 "GND" H 9958 2477 50  0000 L CNN
-F 2 "" H 10100 2450 50  0001 C CNN
+F 2 "TestPoint:TestPoint_Pad_D1.0mm" H 10100 2450 50  0001 C CNN
 F 3 "~" H 10100 2450 50  0001 C CNN
 	1    9900 2450
@@
 F 0 "TP12" H 10308 2568 50  0000 L CNN
 F 1 "GND" H 10308 2477 50  0000 L CNN
-F 2 "" H 10450 2450 50  0001 C CNN
+F 2 "VNA_Footprints:S1751-46_smdTestPoint" H 10450 2450 50  0001 C CNN
 F 3 "~" H 10450 2450 50  0001 C CNN
 	1    10250 2450
@@
 F 0 "TP14" H 10608 2568 50  0000 L CNN
 F 1 "GND" H 10608 2477 50  0000 L CNN
-F 2 "" H 10750 2450 50  0001 C CNN
+F 2 "VNA_Footprints:S1751-46_smdTestPoint" H 10750 2450 50  0001 C CNN
 F 3 "~" H 10750 2450 50  0001 C CNN
 	1    10550 2450
@@
 F 0 "FB4" V 1750 2400 50  0000 C CNN
 F 1 "Bead" V 1850 2700 50  0000 C CNN
-F 2 "" V 1730 2550 50  0001 C CNN
+F 2 "VNA_Footprints:BEADC1608X95N" V 1730 2550 50  0001 C CNN
 F 3 "~" H 1800 2550 50  0001 C CNN
 	1    1800 2550

Commit message: More schematic changes + updated functionals
Parts:
- removed U5: TVL755P, Package_DFN_QFN:DFN-6-1EP_2x2mm_P0.65mm_EP1x1.6mm, symbol VNA_Symbols:TVL755P
- added U5: LP5912, Package_DFN_QFN:DFN-6-1EP_2x2mm_P0.65mm_EP1x1.6mm, symbol VNA_Symbols:LP5912
Changed lines of the file:
@@
 	5150 3950 5150 3800
 Connection ~ 4950 3950
-Text Notes 4000 3550 0    100  ~ 0
+Text Notes 4000 3550 0    100  ~ 6
 1V8 LDO\n
 Wire Wire Line
@@
 	1    0    0    -1
 $EndComp
-Text Notes 1300 2150 0    100  ~ 0
+Text Notes 1300 2150 0    100  ~ 6
 5V (Filtered)
-Text HLabel 3350 3800 1    49   Input ~ 0
+Text HLabel 3350 3800 1    49   Input ~ 6
 3V3A
-Text HLabel 5150 3800 1    49   Input ~ 0
+Text HLabel 5150 3800 1    49   Input ~ 6
 1V8
-Text HLabel 2550 2400 1    49   Input ~ 0
+Text HLabel 2550 2400 1    49   Input ~ 6
 5V0
 Wire Wire Line
@@
 	1    0    0    -1
 $EndComp
-Text Notes 2250 3600 2    100  ~ 0
+Text Notes 2250 3600 2    100  ~ 6
 3V3A LDO
 Wire Wire Line
@@
 Wire Wire Line
 	2550 3950 2850 3950
-Text HLabel 2850 3850 1    49   Input ~ 0
+Text HLabel 2850 3850 1    49   Input ~ 6
 3V3A
 Connection ~ 2550 3950
@@
 $EndComp
 NoConn ~ 2150 4150
-$Comp
-L VNA_Symbols:TVL755P U5
-U 1 1 5CFCC1C6
-P 4200 2700
-F 0 "U5" H 4225 3125 50  0000 C CNN
-F 1 "TVL755P" H 4225 3034 50  0000 C CNN
-F 2 "Package_DFN_QFN:DFN-6-1EP_2x2mm_P0.65mm_EP1x1.6mm" H 4200 3150 100 0001 C CNN
-F 3 "" H 4200 3150 100 0001 C CNN
-	1    4200 2700
-	1    0    0    -1
-$EndComp
-Wire Wire Line
-	3750 2650 3750 2500
-Wire Wire Line
-	3750 2500 3900 2500
-Wire Wire Line
-	3750 2650 3900 2650
+Wire Wire Line
+	3750 2700 3750 2500
 $Comp
 L Device:C C32
@@
 Wire Wire Line
 	4950 2500 5250 2500
-Text HLabel 5250 2400 1    49   Input ~ 0
+Text HLabel 5250 2400 1    49   Input ~ 6
 3V3
 Connection ~ 4950 2500
@@
 $EndComp
 Wire Wire Line
-	4550 2650 4600 2650
-Wire Wire Line
-	4600 2650 4600 2750
-Wire Wire Line
-	4550 2950 4600 2950
-Connection ~ 4600 2950
-Wire Wire Line
-	4600 2950 4600 3050
-Wire Wire Line
-	4550 2850 4600 2850
-Connection ~ 4600 2850
-Wire Wire Line
-	4600 2850 4600 2950
-Wire Wire Line
-	4550 2750 4600 2750
-Connection ~ 4600 2750
-Wire Wire Line
-	4600 2750 4600 2850
+	4550 2700 4600 2700
+Wire Wire Line
+	4600 2700 4600 2800
+Wire Wire Line
+	4550 3000 4600 3000
+Connection ~ 4600 3000
+Wire Wire Line
+	4600 3000 4600 3100
+Wire Wire Line
+	4550 2900 4600 2900
+Connection ~ 4600 2900
+Wire Wire Line
+	4600 2900 4600 3000
+Wire Wire Line
+	4550 2800 4600 2800
+Connection ~ 4600 2800
+Wire Wire Line
+	4600 2800 4600 2900
 $Comp
 L power:GND #PWR037
 U 1 1 5CFD53FA
-P 4600 3050
-F 0 "#PWR037" H 4600 2800 50  0001 C CNN
-F 1 "GND" H 4605 2877 50  0000 C CNN
-F 2 "" H 4600 3050 50  0001 C CNN
-F 3 "" H 4600 3050 50  0001 C CNN
-	1    4600 3050
+P 4600 3100
+F 0 "#PWR037" H 4600 2850 50  0001 C CNN
+F 1 "GND" H 4605 2927 50  0000 C CNN
+F 2 "" H 4600 3100 50  0001 C CNN
+F 3 "" H 4600 3100 50  0001 C CNN
+	1    4600 3100
 	1    0    0    -1
 $EndComp
 Connection ~ 3750 2500
-Text Notes 4600 2200 2    100  ~ 0
+Text Notes 4600 2200 2    100  ~ 6
 3V3 LDO
 $Comp
@@
 	0    1    1    0
 $EndComp
-Text HLabel 1250 1400 0    49   Input ~ 0
+Text HLabel 1250 1400 0    49   Input ~ 6
 VBUS
 Wire Wire Line
 	1900 1400 2200 1400
-Text Label 2300 1400 0    50   ~ 0
+Text Label 2300 1400 0    50   ~ 6
 VIN
-Text Label 1050 2400 1    50   ~ 0
+Text Label 1050 2400 1    50   ~ 6
 VIN
-Text Label 3350 2400 1    50   ~ 0
+Text Label 3350 2400 1    50   ~ 6
 VIN
-Text Label 1100 3850 1    50   ~ 0
+Text Label 1100 3850 1    50   ~ 6
 VIN
-Text Notes 1200 1150 0    100  ~ 0
+Text Notes 1200 1150 0    100  ~ 6
 Input Protection
 Wire Wire Line
@@
 Wire Wire Line
 	6600 2600 6600 2550
-Text HLabel 6600 2550 1    50   Input ~ 0
+Text HLabel 6600 2550 1    50   Input ~ 6
 3V3A
-Text HLabel 6150 3500 0    50   Input ~ 0
+Text HLabel 6150 3500 0    50   Input ~ 6
 1V8
 Wire Wire Line
@@
 	1    0    0    -1
 $EndComp
-Text Notes 6800 2200 0    100  ~ 0
+Text Notes 6800 2200 0    100  ~ 6
 Voltage Rail LEDs
 Wire Wire Line
 	7250 2600 7250 2550
-Text HLabel 7250 2550 1    50   Input ~ 0
+Text HLabel 7250 2550 1    50   Input ~ 6
 3V3A
 Wire Wire Line
@@
 Wire Wire Line
 	7650 2600 7650 2550
-Text HLabel 7650 2550 1    50   Input ~ 0
+Text HLabel 7650 2550 1    50   Input ~ 6
 3V3
 Wire Wire Line
@@
 Wire Wire Line
 	8050 2600 8050 2550
-Text HLabel 8050 2550 1    50   Input ~ 0
+Text HLabel 8050 2550 1    50   Input ~ 6
 5V0
 Wire Wire Line
@@
 	1    0    0    -1
 $EndComp
-Text HLabel 8400 2550 1    49   Input ~ 0
+Text HLabel 8400 2550 1    49   Input ~ 6
 VBUS
 Connection ~ 5150 3950
@@
 	1    0    0    -1
 $EndComp
-Text Notes 9150 2200 0    100  ~ 0
+Text Notes 9150 2200 0    100  ~ 6
 Ground Test Points
 $Comp
@@
 	0    1    1    0
 $EndComp
+$Comp
+L VNA_Symbols:LP5912 U5
+U 1 1 5CAEAD8A
+P 4250 2750
+F 0 "U5" H 4100 3200 49  0000 C CNN
+F 1 "LP5912" H 4200 3100 49  0000 C CNN
+F 2 "Package_DFN_QFN:DFN-6-1EP_2x2mm_P0.65mm_EP1x1.6mm" H 4200 3100 49  0001 C CNN
+F 3 "" H 4200 3100 49  0001 C CNN
+	1    4250 2750
+	1    0    0    -1
+$EndComp
+Wire Wire Line
+	3750 2700 3950 2700
+Wire Wire Line
+	3750 2500 3950 2500
 $EndSCHEMATC
