File: Hardware/Ecal/Ecal.sch (KiCad schematic (older format))
At the start: 18 parts, among them J1 USB_B_Micro, J2 SMA, J3 SMA, U1 LP5912, U2 PE42440

Commit message: phase comp on ad8302 implemented in matlab
Parts:
- U1: symbol VNA_Symbols:LP5912 -> Ecal-rescue:LP5912-VNA_Symbols
Changed lines of the file:
@@
 EESchema Schematic File Version 4
-LIBS:Filter_Bank_Dev_Rev_0-cache
-LIBS:SAO101-cache
+LIBS:Ecal-cache
 EELAYER 29 0
 EELAYER END
@@
 	1050 3225 1050 3275
 $Comp
-L VNA_Symbols:LP5912 U1
+L Ecal-rescue:LP5912-VNA_Symbols U1
 U 1 1 5CFAAA40
 P 1700 3125

Commit message: more thesis progress!
Parts:
- removed U2: PE42440, VNA_Footprints:QFN-16-1EP_3x3mm_P0.5mm_EP2.7x2.7mm_ThermalVias, symbol Ecal-rescue:PE42440-VNA_Symbols
- added U?: PE42440, symbol VNA_Symbols:PE42440
Connections:
- net +3.3VA: now also U?.2 (VCC)
- net GND: now also U?.1 (GND), U?.10 (GND), U?.12 (GND), U?.14 (GND), U?.17 (GND), U?.5 (GND), U?.7 (GND), U?.8 (RF3), U?.9 (GND)
- net IN: now also U?.11 (RFC)
- net LOAD: now also U?.6 (RF4)
- net OPEN: now also U?.13 (RF1)
- net SCL: now also U?.4 (CTRL1)
- net SDA: now also U?.3 (CTRL2)
- net THRU: now also U?.15 (RF2)
Other:
- moved on the sheet: C3, C5, J2, J3
Changed lines of the file:
@@
 EESchema Schematic File Version 4
 LIBS:Ecal-cache
-EELAYER 29 0
+EELAYER 30 0
 EELAYER END
 $Descr A4 11693 8268
@@
 L Connector:Conn_Coaxial J3
 U 1 1 5C2A4464
-P 8975 2750
-F 0 "J3" H 8925 2950 50  0000 L CNN
-F 1 "SMA" H 8875 2850 50  0000 L CNN
-F 2 "VNA_Footprints:SMA_EDGE_MOUNT" H 8975 2750 50  0001 C CNN
-F 3 " ~" H 8975 2750 50  0001 C CNN
-	1    8975 2750
-	1    0    0    -1
-$EndComp
-Wire Wire Line
-	8975 2950 8975 2975
+P 8725 2750
+F 0 "J3" H 8675 2950 50  0000 L CNN
+F 1 "SMA" H 8625 2850 50  0000 L CNN
+F 2 "VNA_Footprints:SMA_EDGE_MOUNT" H 8725 2750 50  0001 C CNN
+F 3 " ~" H 8725 2750 50  0001 C CNN
+	1    8725 2750
+	1    0    0    -1
+$EndComp
+Wire Wire Line
+	8725 2950 8725 2975
 $Comp
 L power:GND #PWR024
 U 1 1 5C2A4626
-P 8975 2975
-F 0 "#PWR024" H 8975 2725 50  0001 C CNN
-F 1 "GND" H 8980 2802 50  0000 C CNN
-F 2 "" H 8975 2975 50  0001 C CNN
-F 3 "" H 8975 2975 50  0001 C CNN
-	1    8975 2975
-	1    0    0    -1
-$EndComp
-$Comp
-L Ecal-rescue:PE42440-VNA_Symbols U2
-U 1 1 5C2A4728
-P 6600 3000
-F 0 "U2" H 7050 3600 50  0000 L CNN
-F 1 "PE42440" H 6800 3500 50  0000 L CNN
-F 2 "VNA_Footprints:QFN-16-1EP_3x3mm_P0.5mm_EP2.7x2.7mm_ThermalVias" H 6300 3500 50  0001 C CNN
-F 3 "" H 6300 3500 50  0001 C CNN
-	1    6600 3000
-	-1   0    0    -1
-$EndComp
-Wire Wire Line
-	6950 3750 6950 3800
-Wire Wire Line
-	6950 3800 6850 3800
-Wire Wire Line
-	6250 3750 6250 3800
-Wire Wire Line
-	6350 3750 6350 3800
-Connection ~ 6350 3800
-Wire Wire Line
-	6350 3800 6250 3800
-Wire Wire Line
-	6450 3750 6450 3800
-Connection ~ 6450 3800
-Wire Wire Line
-	6450 3800 6350 3800
-Wire Wire Line
-	6550 3750 6550 3800
-Connection ~ 6550 3800
-Wire Wire Line
-	6550 3800 6450 3800
-Wire Wire Line
-	6650 3750 6650 3800
-Connection ~ 6650 3800
-Wire Wire Line
-	6650 3800 6550 3800
-Wire Wire Line
-	6750 3750 6750 3800
-Connection ~ 6750 3800
-Wire Wire Line
-	6750 3800 6650 3800
-Wire Wire Line
-	6850 3750 6850 3800
-Connection ~ 6850 3800
-Wire Wire Line
-	6850 3800 6750 3800
+P 8725 2975
+F 0 "#PWR024" H 8725 2725 50  0001 C CNN
+F 1 "GND" H 8730 2802 50  0000 C CNN
+F 2 "" H 8725 2975 50  0001 C CNN
+F 3 "" H 8725 2975 50  0001 C CNN
+	1    8725 2975
+	1    0    0    -1
+$EndComp
+Wire Wire Line
+	6950 3450 6950 3500
+Wire Wire Line
+	6950 3500 6850 3500
+Wire Wire Line
+	6250 3450 6250 3500
+Wire Wire Line
+	6350 3450 6350 3500
+Connection ~ 6350 3500
+Wire Wire Line
+	6350 3500 6250 3500
+Wire Wire Line
+	6450 3450 6450 3500
+Connection ~ 6450 3500
+Wire Wire Line
+	6450 3500 6350 3500
+Wire Wire Line
+	6550 3450 6550 3500
+Connection ~ 6550 3500
+Wire Wire Line
+	6550 3500 6450 3500
+Wire Wire Line
+	6650 3450 6650 3500
+Connection ~ 6650 3500
+Wire Wire Line
+	6650 3500 6550 3500
+Wire Wire Line
+	6750 3450 6750 3500
+Connection ~ 6750 3500
+Wire Wire Line
+	6750 3500 6650 3500
+Wire Wire Line
+	6850 3450 6850 3500
+Connection ~ 6850 3500
+Wire Wire Line
+	6850 3500 6750 3500
 $Comp
 L power:GND #PWR019
 U 1 1 5C2A4744
-P 6250 3800
-F 0 "#PWR019" H 6250 3550 50  0001 C CNN
-F 1 "GND" H 6255 3627 50  0000 C CNN
-F 2 "" H 6250 3800 50  0001 C CNN
-F 3 "" H 6250 3800 50  0001 C CNN
-	1    6250 3800
+P 6250 3500
+F 0 "#PWR019" H 6250 3250 50  0001 C CNN
+F 1 "GND" H 6255 3327 50  0000 C CNN
+F 2 "" H 6250 3500 50  0001 C CNN
+F 3 "" H 6250 3500 50  0001 C CNN
+	1    6250 3500
 	-1   0    0    -1
 $EndComp
-Connection ~ 6250 3800
-NoConn ~ 6150 3750
+Connection ~ 6250 3500
+NoConn ~ 6150 3450
 $Comp
 L Device:C C3
 U 1 1 5C2A474C
-P 5275 2650
-F 0 "C3" V 5125 2650 50  0000 C CNN
-F 1 "1n" V 5425 2650 50  0000 C CNN
-F 2 "Capacitor_SMD:C_0402_1005Metric" H 5313 2500 50  0001 C CNN
-F 3 "~" H 5275 2650 50  0001 C CNN
-	1    5275 2650
+P 5425 2650
+F 0 "C3" V 5275 2650 50  0000 C CNN
+F 1 "1n" V 5575 2650 50  0000 C CNN
+F 2 "Capacitor_SMD:C_0402_1005Metric" H 5463 2500 50  0001 C CNN
+F 3 "~" H 5425 2650 50  0001 C CNN
+	1    5425 2650
 	0    1    1    0
 $EndComp
@@
 L Connector:Conn_Coaxial J2
 U 1 1 5C2A4764
-P 4825 2650
-F 0 "J2" H 4875 2850 50  0000 L CNN
-F 1 "SMA" H 4825 2750 50  0000 L CNN
-F 2 "VNA_Footprints:SMA_EDGE_MOUNT" H 4825 2650 50  0001 C CNN
-F 3 " ~" H 4825 2650 50  0001 C CNN
-	1    4825 2650
+P 4975 2650
+F 0 "J2" H 5025 2850 50  0000 L CNN
+F 1 "SMA" H 4975 2750 50  0000 L CNN
+F 2 "VNA_Footprints:SMA_EDGE_MOUNT" H 4975 2650 50  0001 C CNN
+F 3 " ~" H 4975 2650 50  0001 C CNN
+	1    4975 2650
 	-1   0    0    -1
 $EndComp
 Wire Wire Line
-	4825 2850 4825 2950
+	4975 2850 4975 2900
 $Comp
 L power:GND #PWR018
 U 1 1 5C2A476C
-P 4825 2950
-F 0 "#PWR018" H 4825 2700 50  0001 C CNN
-F 1 "GND" H 4830 2777 50  0000 C CNN
-F 2 "" H 4825 2950 50  0001 C CNN
-F 3 "" H 4825 2950 50  0001 C CNN
-	1    4825 2950
+P 4975 2900
+F 0 "#PWR018" H 4975 2650 50  0001 C CNN
+F 1 "GND" H 4980 2727 50  0000 C CNN
+F 2 "" H 4975 2900 50  0001 C CNN
+F 3 "" H 4975 2900 50  0001 C CNN
+	1    4975 2900
 	-1   0    0    -1
 $EndComp
@@
 	6500 2050 6500 2200
 Wire Wire Line
-	5025 2650 5125 2650
-Wire Wire Line
-	5425 2650 5850 2650
+	5175 2650 5275 2650
+Wire Wire Line
+	5575 2650 5850 2650
 $Comp
 L Device:C C4
@@
 	1    0    0    -1
 $EndComp
-Text Notes 4375 2700 0    50   ~ 0
+Text Notes 4800 2400 0    50   ~ 0
 PORT 1
-Text Notes 9125 2800 0    50   ~ 0
+Text Notes 8600 2500 0    50   ~ 0
 PORT 2
 Text Label 7675 2750 2    50   ~ 0
@@
 $EndComp
 Wire Wire Line
-	7300 3150 7675 3150
-Wire Wire Line
-	7300 3250 7675 3250
-Text Label 7675 3150 2    50   ~ 0
+	5850 2950 5600 2950
+Wire Wire Line
+	5850 2850 5600 2850
+Text Label 5600 2950 0    50   ~ 0
 SDA
-Text Label 7675 3250 2    50   ~ 0
+Text Label 5600 2850 0    50   ~ 0
 SCL
 $Comp
 L Device:C C5
 U 1 1 5D1271E4
-P 8350 2750
-F 0 "C5" V 8200 2750 50  0000 C CNN
-F 1 "1n" V 8500 2750 50  0000 C CNN
-F 2 "Capacitor_SMD:C_0402_1005Metric" H 8388 2600 50  0001 C CNN
-F 3 "~" H 8350 2750 50  0001 C CNN
-	1    8350 2750
+P 8300 2750
+F 0 "C5" V 8150 2750 50  0000 C CNN
+F 1 "1n" V 8450 2750 50  0000 C CNN
+F 2 "Capacitor_SMD:C_0402_1005Metric" H 8338 2600 50  0001 C CNN
+F 3 "~" H 8300 2750 50  0001 C CNN
+	1    8300 2750
 	0    1    1    0
 $EndComp
 Wire Wire Line
-	7300 2750 8200 2750
-Wire Wire Line
-	8500 2750 8775 2750
-Text Notes 7225 4250 0    50   ~ 0
+	7300 2750 8150 2750
+Wire Wire Line
+	8450 2750 8525 2750
+Text Notes 7025 4775 0    50   ~ 0
 NOTE: SDA and SCL are named as\nmicrocontroller can be configured\nto talk over I2C on these pins, will \nhowever be configured as GPIO as \nonly two pins required.
-Text Notes 6250 1700 0    100  ~ 0
+Text Notes 6200 1400 0    100  ~ 0
 RF Switch
 Text Label 5600 2650 0    50   ~ 0
 IN
+$Comp
+L VNA_Symbols:PE42440 U?
+U 1 1 5DA1D073
+P 6600 3000
+F 0 "U?" H 7100 3575 50  0000 C CNN
+F 1 "PE42440" H 6975 3500 50  0000 C CNN
+F 2 "" H 6300 3500 50  0001 C CNN
+F 3 "" H 6300 3500 50  0001 C CNN
+	1    6600 3000
+	-1   0    0    -1
+$EndComp
 $EndSCHEMATC
